File: Hardware/Source-files/TWV.brd (EAGLE design)
At the start: 49.5 x 72.5 mm, 66 parts, among them T10 TEST_POINT_2MM, T11 TEST_POINT_2MM, T3 TEST_POINT_2MM, T4 TEST_POINT_2MM, T5 TEST_POINT_2MM, T6 TEST_POINT_2MM, T9 TEST_POINT_2MM

Commit message: Stable PCB version
Parts:
- removed C11: 2.2uF, Capacitor:0603
- removed C9: 10uF, Capacitor:0603
- removed R10: 150k, Resistors:0603
- removed R19: 47k, Resistors:0603
- removed XS5: BM02B-SRSS-TB, Connectors:BM02B-SRSS-TB
- added C12: 10uF, Capacitor:0603
- added VD10: SD103CW-AQ, Diode:SOD-123F
- added VD2, VD6: SD0805S040S0R5, Diode:0805
- added VT2: SI2333, Transistor:SOT-23
- added VT3: IRLML6401, Transistor:SOT-23
- C7: value 1 uF -> 0.47 uF
- D1: value 150060RS75000 -> BL-HKC37A-AV-TRB
- D4: value 150060RS75000 -> BL-HB337A-AV-TRB
- DD3: value NPM1300 -> TPS64201DBVR; device Power-IC:QFN32-5X5MM -> Power-IC:SOT23-6
- R12, R3, R6, R8: value 39 -> 330
- R23: value 0 -> 360 kOhm; device Resistors:0805 -> Resistors:0603
- R24: value 4.7k -> 620 kOhm
- R25: value 4.7k -> 33 mOhm
- moved C7 15.0 mm to (12.4, 18.9), turned to 180 degrees
- moved R23 13.5 mm to (10.1, 24.4)
- moved C5 12.7 mm to (40.2, 32.2), flipped to the bottom, turned to 270 degrees
- moved R25 8.49 mm to (15.7, 25.9), turned to 270 degrees
- moved L1 7.79 mm to (17.6, 19.9), turned to 270 degrees
- moved C8 6.93 mm to (32.5, 34.1), flipped to the bottom, turned to 270 degrees
- moved C13 6.71 mm to (39.4, 38.5), flipped to the bottom, turned to 0 degrees
- moved R24 5.95 mm to (12.3, 23.6), turned to 0 degrees
- moved C4 4.96 mm to (40.3, 35.7), flipped to the bottom, turned to 180 degrees
- moved R5 4.30 mm to (39.7, 44.9)
- moved R2 4.30 mm to (42.5, 44.9)
- moved R4 4.30 mm to (41.3, 44.9)
- moved R22 3.24 mm to (41.3, 41.1)
- moved R16 2.67 mm to (39.4, 41.2)
- moved C2 2.57 mm to (38.1, 41.2)
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Connections:
- removed net CC1: DD3.23, R7.2, XS7.A5
- removed net CC2: DD3.24, R11.2, XS7.B5
- removed net N$4: DD3.16, R19.1
- removed net N1: DD3.1, L1.P$2
- removed net SCL: DD1.18, DD3.14, R25.2
- removed net SDA: DD1.19, DD3.13, R24.2
- removed net VBUSOUT: C14.1, DD1.22, DD3.22
- removed net VSYS: DD3.20, DD3.30, DD3.4
- new net N$2: VT3.3, XS4.1
- new net N$22: L1.P$1, VD10.C, VT2.3
- new net N$23: DD3.6, VT2.1
- new net N$25: DD3.4, R25.2, VT2.2
- new net N$26: DD3.3, R23.2, R24.1
- new net N$7: R7.2, XS7.A5
- net +3.3V: now also C7.1, L1.P$2, R24.2; no longer R23.1, R24.1, R25.1
- net GND: now also C12.2, DD3.1, R23.1, VD10.A, VT3.1, XS4.2; no longer C11.2, C9.2, DD3.33, R10.2, R19.2, XS4.1, XS5.2
- net N$3: now also R11.2, XS7.B5; no longer DD3.17, R10.1
- net VBAT: now also VD6.1, VT3.2; no longer C11.1, DD3.19, XS4.2
- net VBUS: now also C14.1, DD1.22, VD2.1; no longer C7.1, DD3.21, XS5.1
- net VOUT: now also C12.1, DD3.5, R25.1, VD2.2, VD6.2; no longer C9.1, DD3.12, DD3.3, L1.P$1, R23.2
Routing:
- net CC1: track 54.3 -> 0.00 mm, vias 3 -> 0
- net CC2: track 47.8 -> 0.00 mm, vias 3 -> 0
- net SCL: track 30.1 -> 0.00 mm, vias 5 -> 0
- net SDA: track 30.0 -> 0.00 mm, vias 4 -> 0
- net VBUSOUT: track 22.4 -> 0.00 mm, vias 2 -> 0
- net VSYS: track 18.1 -> 0.00 mm, vias 3 -> 0
- net N$7: track 0.00 -> 12.0 mm, vias 0 -> 2
- net VOUT: track 21.5 -> 9.92 mm, vias 2 -> 0
- net VBUS: track 53.8 -> 63.7 mm, vias 0 -> 1
- net N$3: track 3.41 -> 12.0 mm, vias 0 -> 2
- net CONTROL2: track 6.59 -> 13.2 mm, vias 0 -> 1
- net N$23: track 0.00 -> 6.55 mm
- net CONTROL: track 9.59 -> 14.4 mm, vias 2 -> 1
- net XS2.1: track 64.3 -> 59.6 mm
- net N$25: track 0.00 -> 4.24 mm
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- removed copper zone on layer 1, net N1
- removed copper zone on layer 1, net VOUT
Other:
- outline, holes or cut-outs redrawn
